File: Hardware/TempControler/Power.sch (KiCad schematic (older format))
At the start: 0 parts

Commit message: Schematic Complete
DRC - Done
Schematic - Done
Values - Done
Part Selection - In Progress
Footprint assignment- In Progress
Parts:
- added BT1: Battery, symbol Device:Battery
- added C4, C6: 470uF, Capacitor_SMD:CP_Elec_10x10, symbol Device:CP
- added C5: 470pF, Capacitor_SMD:C_0603_1608Metric, symbol Device:C
- added C7: 100uF, Capacitor_SMD:CP_Elec_6.3x5.8, symbol Device:CP
- added D1, D2: D_Schottky, Diode_SMD:D_SOD-128, symbol Device:D_Schottky
- added L1: 100uH, Inductor_THT:L_Toroid_Vertical_L13.0mm_W6.5mm_P5.60mm, symbol Device:L_Core_Iron
- added L2: 1uH, Inductor_THT:L_Toroid_Vertical_L13.0mm_W6.5mm_P5.60mm, symbol Device:L_Core_Iron
- added R4, R5: 10k, Resistor_SMD:R_0603_1608Metric, symbol Device:R
- added R6: .1, Resistor_SMD:R_1206_3216Metric, symbol Device:R
- added R7: 22.1k, Resistor_SMD:R_0603_1608Metric, symbol Device:R
- added R8: 36k, Resistor_SMD:R_0603_1608Metric, symbol Device:R
- added U3: AP34063S8L-13, Package_SO:SO-8_3.9x4.9mm_P1.27mm, symbol Regulator_Switching:MC34063AD
Connections:
- new net: R6.1, U3.1 (SwC), U3.7 (Ipk), U3.8 (DC)
- new net: D2.1 (K), L1.1, U3.2 (SwE)
- new net: C5.1, U3.3 (TC)
- new net: R7.1, R8.2, U3.5 (Vfb)
- new net: C6.1, L1.2, L2.1, R8.1
- new net: BT1.1 (+), D1.2 (A), R4.1
- new net +24V: C4.1, D1.1 (K), R6.2, U3.6 (Vin)
- new net +3V3: C7.1, L2.2
- new net GND: BT1.2 (-), C4.2, C5.2, C6.2, C7.2, D2.2 (A), R5.2, R7.2, U3.4 (GND)
- new net bSence: R4.2, R5.1

Commit message: All Part Numbers Selected
Next step select all footprints
Parts:
- BT1: footprint (none) -> Connector_PinHeader_1.27mm:PinHeader_1x02_P1.27mm_Vertical; Mouser (none) -> N/A
- C4, C6: Mouser (none) -> 647-UUR1E471MNL1GS
- C5: Mouser (none) -> 80-C0603C471J5G
- C7: Mouser (none) -> 140-VZS101M1ETR0606
- D1, D2: value D_Schottky -> RB080LAM-30TR; Mouser (none) -> 755-RB080LAM-30TR
- L1, L2: Mouser (none) -> Hand Made
- R4, R5: Mouser (none) -> 667-ERJ-3EKF1002V
- R6: Mouser (none) -> 71-CRCW1206J-0.1-E3
- R7: Mouser (none) -> 603-RC0603FR-1022K1L
- R8: Mouser (none) -> 667-ERJ-3EKF3602V
Changed lines of the file:
@@
 F 1 "470uF" H 3218 2305 50  0000 L CNN
 F 2 "Capacitor_SMD:CP_Elec_10x10" H 3138 2200 50  0001 C CNN
-F 3 "~" H 3100 2350 50  0001 C CNN
+F 3 "https://www.mouser.com/datasheet/2/293/e_uur-880111.pdf" H 3100 2350 50  0001 C CNN
+F 4 "647-UUR1E471MNL1GS" H 3100 2350 50  0001 C CNN "Mouser"
 	1    3100 2350
 	1    0    0    -1
@@
 F 1 ".1" V 3984 1850 50  0000 C CNN
 F 2 "Resistor_SMD:R_1206_3216Metric" V 4030 1850 50  0001 C CNN
-F 3 "~" H 4100 1850 50  0001 C CNN
+F 3 "https://www.mouser.com/datasheet/2/427/dcrcwe3-1762152.pdf" H 4100 1850 50  0001 C CNN
+F 4 "71-CRCW1206J-0.1-E3" H 4100 1850 50  0001 C CNN "Mouser"
 	1    4100 1850
 	0    1    1    0
@@
 F 1 "470pF" H 3665 2705 50  0000 L CNN
 F 2 "Capacitor_SMD:C_0603_1608Metric" H 3588 2600 50  0001 C CNN
-F 3 "~" H 3550 2750 50  0001 C CNN
+F 3 "https://www.mouser.com/datasheet/2/212/KEM_C1003_C0G_SMD-1101588.pdf" H 3550 2750 50  0001 C CNN
+F 4 "80-C0603C471J5G" H 3550 2750 50  0001 C CNN "Mouser"
 	1    3550 2750
 	1    0    0    -1
@@
 P 4700 2750
 F 0 "D2" V 4700 2830 50  0000 L CNN
-F 1 "D_Schottky" V 4745 2830 50  0001 L CNN
+F 1 "RB080LAM-30TR" V 4745 2830 50  0001 L CNN
 F 2 "Diode_SMD:D_SOD-128" H 4700 2750 50  0001 C CNN
-F 3 "~" H 4700 2750 50  0001 C CNN
+F 3 "https://www.mouser.com/datasheet/2/348/rb080lam_30tr_e-1869813.pdf" H 4700 2750 50  0001 C CNN
+F 4 "755-RB080LAM-30TR" H 4700 2750 50  0001 C CNN "Mouser"
 	1    4700 2750
 	0    1    1    0
@@
 F 1 "100uH" H 5138 2705 50  0000 L CNN
 F 2 "Inductor_THT:L_Toroid_Vertical_L13.0mm_W6.5mm_P5.60mm" H 5050 2750 50  0001 C CNN
-F 3 "~" H 5050 2750 50  0001 C CNN
+F 3 "N/A" H 5050 2750 50  0001 C CNN
+F 4 "Hand Made" H 5050 2750 50  0001 C CNN "Mouser"
 	1    5050 2750
 	1    0    0    -1
@@
 F 1 "22.1k" V 4234 3400 50  0000 C CNN
 F 2 "Resistor_SMD:R_0603_1608Metric" V 4280 3400 50  0001 C CNN
-F 3 "~" H 4350 3400 50  0001 C CNN
+F 3 "https://www.mouser.com/datasheet/2/447/Yageo_03_18_2021_PYu_RC_Group_51_RoHS_L_11-2199992.pdf" H 4350 3400 50  0001 C CNN
+F 4 "603-RC0603FR-1022K1L" H 4350 3400 50  0001 C CNN "Mouser"
 	1    4350 3400
 	0    1    1    0
@@
 F 1 "36k" V 4634 3400 50  0000 C CNN
 F 2 "Resistor_SMD:R_0603_1608Metric" V 4680 3400 50  0001 C CNN
-F 3 "~" H 4750 3400 50  0001 C CNN
+F 3 "https://www.mouser.com/datasheet/2/315/AOA0000C304-1149620.pdf" H 4750 3400 50  0001 C CNN
+F 4 "667-ERJ-3EKF3602V" H 4750 3400 50  0001 C CNN "Mouser"
 	1    4750 3400
 	0    1    1    0
@@
 F 1 "470uF" H 5168 3555 50  0000 L CNN
 F 2 "Capacitor_SMD:CP_Elec_10x10" H 5088 3450 50  0001 C CNN
-F 3 "~" H 5050 3600 50  0001 C CNN
+F 3 "https://www.mouser.com/datasheet/2/293/e_uur-880111.pdf" H 5050 3600 50  0001 C CNN
+F 4 "647-UUR1E471MNL1GS" H 5050 3600 50  0001 C CNN "Mouser"
 	1    5050 3600
 	1    0    0    -1
@@
 F 1 "1uH" V 5434 3400 50  0000 C CNN
 F 2 "Inductor_THT:L_Toroid_Vertical_L13.0mm_W6.5mm_P5.60mm" H 5300 3400 50  0001 C CNN
-F 3 "~" H 5300 3400 50  0001 C CNN
+F 3 "N/A" H 5300 3400 50  0001 C CNN
+F 4 "Hand Made" H 5300 3400 50  0001 C CNN "Mouser"
 	1    5300 3400
 	0    -1   -1   0
@@
 F 1 "100uF" H 5668 3555 50  0000 L CNN
 F 2 "Capacitor_SMD:CP_Elec_6.3x5.8" H 5588 3450 50  0001 C CNN
-F 3 "~" H 5550 3600 50  0001 C CNN
+F 3 "https://www.mouser.com/datasheet/2/231/161587298653-2307449.pdf" H 5550 3600 50  0001 C CNN
+F 4 "140-VZS101M1ETR0606" H 5550 3600 50  0001 C CNN "Mouser"
 	1    5550 3600
 	1    0    0    -1
@@
 F 0 "BT1" H 2808 2946 50  0000 L CNN
 F 1 "Battery" H 2808 2855 50  0001 L CNN
-F 2 "" V 2700 2960 50  0001 C CNN
-F 3 "~" V 2700 2960 50  0001 C CNN
+F 2 "Connector_PinHeader_1.27mm:PinHeader_1x02_P1.27mm_Vertical" V 2700 2960 50  0001 C CNN
+F 3 "N/A" V 2700 2960 50  0001 C CNN
+F 4 "N/A" H 2700 2900 50  0001 C CNN "Mouser"
 	1    2700 2900
 	1    0    0    -1
@@
 P 2700 2400
 F 0 "D1" V 2654 2480 50  0000 L CNN
-F 1 "D_Schottky" V 2745 2480 50  0001 L CNN
+F 1 "RB080LAM-30TR" V 2745 2480 50  0001 L CNN
 F 2 "Diode_SMD:D_SOD-128" H 2700 2400 50  0001 C CNN
-F 3 "~" H 2700 2400 50  0001 C CNN
+F 3 "https://www.mouser.com/datasheet/2/348/rb080lam_30tr_e-1869813.pdf" H 2700 2400 50  0001 C CNN
+F 4 "755-RB080LAM-30TR" H 2700 2400 50  0001 C CNN "Mouser"
 	1    2700 2400
 	0    1    1    0
@@
 F 1 "10k" H 2470 2755 50  0000 L CNN
 F 2 "Resistor_SMD:R_0603_1608Metric" V 2330 2800 50  0001 C CNN
-F 3 "~" H 2400 2800 50  0001 C CNN
+F 3 "https://www.mouser.com/datasheet/2/315/AOA0000C304-1149620.pdf" H 2400 2800 50  0001 C CNN
+F 4 "667-ERJ-3EKF1002V" H 2400 2800 50  0001 C CNN "Mouser"
 	1    2400 2800
 	1    0    0    -1
@@
 F 1 "10k" H 2470 3155 50  0000 L CNN
 F 2 "Resistor_SMD:R_0603_1608Metric" V 2330 3200 50  0001 C CNN
-F 3 "~" H 2400 3200 50  0001 C CNN
+F 3 "https://www.mouser.com/datasheet/2/315/AOA0000C304-1149620.pdf" H 2400 3200 50  0001 C CNN
+F 4 "667-ERJ-3EKF1002V" H 2400 3200 50  0001 C CNN "Mouser"
 	1    2400 3200
 	1    0    0    -1
