File: Hardware/TempControler/Thermostat.sch (KiCad schematic (older format))
At the start: 22 parts, among them J2 Conn_01x12_Male

Commit message: All Part Numbers Selected
Next step select all footprints
Parts:
- C10, C11: Mouser (none) -> 80-C0805C104K5R
- D10, D4: Mouser (none) -> 621-RDBF32-13
- D16, D18: value D_Schottky -> RB080LAM-30TR; Mouser (none) -> 755-RB080LAM-30TR
- D17, D19: Mouser (none) -> 755-BZX84C3V0LFHT116
- J2: Mouser (none) -> 490-TBL00150012GY2GY
- R11, R12: value 57k -> 56k; Mouser (none) -> 791-RMC16K563FTP
Changed lines of the file:
@@
 F 1 "Conn_01x12_Male" H 908 2690 50  0000 C CNN
 F 2 "" H 800 2100 50  0001 C CNN
-F 3 "~" H 800 2100 50  0001 C CNN
+F 3 "https://www.mouser.com/datasheet/2/670/tbl001_500-1609255.pdf" H 800 2100 50  0001 C CNN
+F 4 "490-TBL00150012GY2GY" H 800 2100 50  0001 C CNN "Mouser"
 	1    800  2100
 	1    0    0    -1
@@
 F 1 "D_Bridge_+-AA" H 2594 1055 50  0001 L CNN
 F 2 "" H 2250 1100 50  0001 C CNN
-F 3 "~" H 2250 1100 50  0001 C CNN
+F 3 "https://www.mouser.com/datasheet/2/115/DIOD_S_A0005424863_1-2542538.pdf" H 2250 1100 50  0001 C CNN
+F 4 "621-RDBF32-13" H 2250 1100 50  0001 C CNN "Mouser"
 	1    2250 1100
 	1    0    0    -1
@@
 F 1 "D_Bridge_+-AA" H 4294 1055 50  0001 L CNN
 F 2 "" H 3950 1100 50  0001 C CNN
-F 3 "~" H 3950 1100 50  0001 C CNN
+F 3 "https://www.mouser.com/datasheet/2/115/DIOD_S_A0005424863_1-2542538.pdf" H 3950 1100 50  0001 C CNN
+F 4 "621-RDBF32-13" H 3950 1100 50  0001 C CNN "Mouser"
 	1    3950 1100
 	1    0    0    -1
@@
 P 5850 1050
 F 0 "R11" V 5643 1050 50  0000 C CNN
-F 1 "57k" V 5734 1050 50  0000 C CNN
+F 1 "56k" V 5734 1050 50  0000 C CNN
 F 2 "Resistor_SMD:R_0603_1608Metric" V 5780 1050 50  0001 C CNN
-F 3 "~" H 5850 1050 50  0001 C CNN
+F 3 "https://www.mouser.com/datasheet/2/210/kamaya_products_RMC__english_20170424_100617-1524908.pdf" H 5850 1050 50  0001 C CNN
+F 4 "791-RMC16K563FTP" H 5850 1050 50  0001 C CNN "Mouser"
 	1    5850 1050
 	0    1    1    0
@@
 P 6450 1800
 F 0 "R12" V 6650 1800 50  0000 C CNN
-F 1 "57k" V 6550 1800 50  0000 C CNN
+F 1 "56k" V 6550 1800 50  0000 C CNN
 F 2 "Resistor_SMD:R_0603_1608Metric" V 6380 1800 50  0001 C CNN
-F 3 "~" H 6450 1800 50  0001 C CNN
+F 3 "https://www.mouser.com/datasheet/2/210/kamaya_products_RMC__english_20170424_100617-1524908.pdf" H 6450 1800 50  0001 C CNN
+F 4 "791-RMC16K563FTP" H 6450 1800 50  0001 C CNN "Mouser"
 	1    6450 1800
 	0    1    1    0
@@
 P 5450 1050
 F 0 "D16" H 5450 925 50  0000 C CNN
-F 1 "D_Schottky" H 5450 924 50  0001 C CNN
+F 1 "RB080LAM-30TR" H 5450 924 50  0001 C CNN
 F 2 "Diode_SMD:D_SOD-128" H 5450 1050 50  0001 C CNN
-F 3 "~" H 5450 1050 50  0001 C CNN
+F 3 "https://www.mouser.com/datasheet/2/348/rb080lam_30tr_e-1869813.pdf" H 5450 1050 50  0001 C CNN
+F 4 "755-RB080LAM-30TR" H 5450 1050 50  0001 C CNN "Mouser"
 	1    5450 1050
 	-1   0    0    1
@@
 P 6050 1800
 F 0 "D18" H 6050 1950 50  0000 C CNN
-F 1 "D_Schottky" H 6050 1674 50  0001 C CNN
+F 1 "RB080LAM-30TR" H 6050 1674 50  0001 C CNN
 F 2 "Diode_SMD:D_SOD-128" H 6050 1800 50  0001 C CNN
-F 3 "~" H 6050 1800 50  0001 C CNN
+F 3 "https://www.mouser.com/datasheet/2/348/rb080lam_30tr_e-1869813.pdf" H 6050 1800 50  0001 C CNN
+F 4 "755-RB080LAM-30TR" H 6050 1800 50  0001 C CNN "Mouser"
 	1    6050 1800
 	-1   0    0    1
@@
 F 1 ".1uF" H 6565 1205 50  0000 L CNN
 F 2 "Capacitor_SMD:C_0805_2012Metric" H 6488 1100 50  0001 C CNN
-F 3 "~" H 6450 1250 50  0001 C CNN
+F 3 "https://www.mouser.com/datasheet/2/212/KEM_C1002_X7R_SMD-1102033.pdf" H 6450 1250 50  0001 C CNN
+F 4 "80-C0805C104K5R" H 6450 1250 50  0001 C CNN "Mouser"
 	1    6450 1250
 	1    0    0    -1
@@
 F 1 ".1uF" H 7165 1955 50  0000 L CNN
 F 2 "Capacitor_SMD:C_0805_2012Metric" H 7088 1850 50  0001 C CNN
-F 3 "~" H 7050 2000 50  0001 C CNN
+F 3 "https://www.mouser.com/datasheet/2/212/KEM_C1002_X7R_SMD-1102033.pdf" H 7050 2000 50  0001 C CNN
+F 4 "80-C0805C104K5R" H 7050 2000 50  0001 C CNN "Mouser"
 	1    7050 2000
 	1    0    0    -1
@@
 F 1 "3V" V 6095 1330 50  0000 L CNN
 F 2 "Diode_SMD:D_SOD-128" H 6050 1250 50  0001 C CNN
-F 3 "~" H 6050 1250 50  0001 C CNN
+F 3 "https://www.mouser.com/datasheet/2/348/ROHM_S_A0010444872_1-2563195.pdf" H 6050 1250 50  0001 C CNN
+F 4 "755-BZX84C3V0LFHT116" H 6050 1250 50  0001 C CNN "Mouser"
 	1    6050 1250
 	0    1    1    0
@@
 F 1 "3V" V 6745 2080 50  0000 L CNN
 F 2 "Diode_SMD:D_SOD-128" H 6700 2000 50  0001 C CNN
-F 3 "~" H 6700 2000 50  0001 C CNN
+F 3 "https://www.mouser.com/datasheet/2/348/ROHM_S_A0010444872_1-2563195.pdf" H 6700 2000 50  0001 C CNN
+F 4 "755-BZX84C3V0LFHT116" H 6700 2000 50  0001 C CNN "Mouser"
 	1    6700 2000
 	0    1    1    0

Commit message: Footprints selected
On to board design
Parts:
- D10, D4: footprint (none) -> Package_DBF:DBF-4
- J2: footprint (none) -> Terminal_Block:TerminalBlock_CUI-12_P5mm
Changed lines of the file:
@@
 F 0 "J2" H 908 2781 50  0000 C CNN
 F 1 "Conn_01x12_Male" H 908 2690 50  0000 C CNN
-F 2 "" H 800 2100 50  0001 C CNN
+F 2 "Terminal_Block:TerminalBlock_CUI-12_P5mm" H 800 2100 50  0001 C CNN
 F 3 "https://www.mouser.com/datasheet/2/670/tbl001_500-1609255.pdf" H 800 2100 50  0001 C CNN
 F 4 "490-TBL00150012GY2GY" H 800 2100 50  0001 C CNN "Mouser"
@@
 F 0 "D4" H 2200 1100 50  0000 L CNN
 F 1 "D_Bridge_+-AA" H 2594 1055 50  0001 L CNN
-F 2 "" H 2250 1100 50  0001 C CNN
+F 2 "Package_DBF:DBF-4" H 2250 1100 50  0001 C CNN
 F 3 "https://www.mouser.com/datasheet/2/115/DIOD_S_A0005424863_1-2542538.pdf" H 2250 1100 50  0001 C CNN
 F 4 "621-RDBF32-13" H 2250 1100 50  0001 C CNN "Mouser"
@@
 F 0 "D10" H 3900 1100 50  0000 L CNN
 F 1 "D_Bridge_+-AA" H 4294 1055 50  0001 L CNN
-F 2 "" H 3950 1100 50  0001 C CNN
+F 2 "Package_DBF:DBF-4" H 3950 1100 50  0001 C CNN
 F 3 "https://www.mouser.com/datasheet/2/115/DIOD_S_A0005424863_1-2542538.pdf" H 3950 1100 50  0001 C CNN
 F 4 "621-RDBF32-13" H 3950 1100 50  0001 C CNN "Mouser"
